File: Schematics/Output Schematics/Output Schematics.kicad_sch (KiCad schematic)
At the start: 11 parts, among them J1 NJ3FD-V, SW1 SW_SPST, U1 TL072, U2 TL072

Commit message: kicad
Parts:
- added U3: MCP4902, symbol Analog_DAC:MCP4902
Connections:
- net Vdd: now also U3.1 (Vdd)
- net DAC0: no longer names the net of R3.2
- net DAC0: now also U3.14 (VA)
- net DAC1: no longer names the net of R4.2
- net DAC1: now also U3.10 (VB)
- new net Arduino_PIN10: U3.3 (~{CS})
- new net Arduino_PIN7: U3.8 (~{LDAC})
- new net Arduino_SCK: U3.4 (SCK)
- new net Arduino_SDA: U3.5 (SDI)
Other:
- note added: "Ring can go to signal or ground depending on what we choose Signal for stereo sound and Ground for Mono"
- note removed: "Ring can go to signal or ground depending on what we choose"
- moved on the sheet: J1, R1, R2, R3, R4, R5, R6, R7, SW1, U1A, U2A

Commit message: commit
Parts:
- R1: renamed from R3; value R -> 10k
- R1: renamed from R2; value R -> 10k
- R1: value R -> 10k
- R1: renamed from R4; value R -> 10k
- R3: renamed from R5; value R -> 20k
- R3: renamed from R7; value =R5 -> 20k
- renumbered R6 to R4
Changed lines of the file:
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@@
 		(dnp no)
 		(fields_autoplaced yes)
-		(property "Reference" "R6"
+		(property "Reference" "R4"
 			(at 209.55 74.93 90)
 			(effects
@@
 			(project "Output Schematics"
 				(path "/1f52c9a4-f58e-4d91-9410-99eb02bd9a97"
-					(reference "R6")
+					(reference "R4")
 					(unit 1)
 				)
@@
 		(dnp no)
 		(fields_autoplaced yes)
-		(property "Reference" "R3"
+		(property "Reference" "R1"
 			(at 147.32 85.09 90)
 			(effects
@@
 			)
 		)
-		(property "Value" "R"
+		(property "Value" "10k"
 			(at 147.32 87.63 90)
 			(effects
@@
 			(project "Output Schematics"
 				(path "/1f52c9a4-f58e-4d91-9410-99eb02bd9a97"
-					(reference "R3")
+					(reference "R1")
 					(unit 1)
 				)
@@
 		(dnp no)
 		(fields_autoplaced yes)
-		(property "Reference" "R2"
+		(property "Reference" "R1"
 			(at 158.75 105.4099 0)
 			(effects
@@
 			)
 		)
-		(property "Value" "R"
+		(property "Value" "10k"
 			(at 158.75 107.9499 0)
 			(effects
@@
 			(project "Output Schematics"
 				(path "/1f52c9a4-f58e-4d91-9410-99eb02bd9a97"
-					(reference "R2")
+					(reference "R1")
 					(unit 1)
 				)
@@
 			)
 		)
-		(property "Value" "R"
+		(property "Value" "10k"
 			(at 167.64 74.93 90)
 			(effects
@@
 		(dnp no)
 		(fields_autoplaced yes)
-		(property "Reference" "R5"
+		(property "Reference" "R3"
 			(at 189.23 87.63 90)
 			(effects
@@
 			)
 		)
-		(property "Value" "R"
+		(property "Value" "20k"
 			(at 189.23 90.17 90)
 			(effects
@@
 			(project "Output Schematics"
 				(path "/1f52c9a4-f58e-4d91-9410-99eb02bd9a97"
-					(reference "R5")
+					(reference "R3")
 					(unit 1)
 				)
@@
 		(on_board yes)
 		(dnp no)
-		(property "Reference" "R4"
+		(property "Reference" "R1"
 			(at 145.034 101.854 90)
 			(effects
@@
 			)
 		)
-		(property "Value" "R"
+		(property "Value" "10k"
 			(at 144.78 99.822 90)
 			(effects
@@
 			(project "Output Schematics"
 				(path "/1f52c9a4-f58e-4d91-9410-99eb02bd9a97"
-					(reference "R4")
+					(reference "R1")
 					(unit 1)
 				)
@@
 		(dnp no)
 		(fields_autoplaced yes)
-		(property "Reference" "R7"
+		(property "Reference" "R3"
 			(at 189.23 77.47 90)
 			(effects
@@
 			)
 		)
-		(property "Value" "=R5"
+		(property "Value" "20k"
 			(at 189.23 80.01 90)
 			(effects
@@
 			(project "Output Schematics"
 				(path "/1f52c9a4-f58e-4d91-9410-99eb02bd9a97"
-					(reference "R7")
-					(unit 1)
-				)
+					(reference "R3")
+					(unit 1)
+				)
